Commit message: Change mesh file names

File: urdf/multicontact/daeun/bridge_1.urdf (robot description, URDF)
Before this commit: robot bridge_1, 1 links, 0 joints
Links:
- link base_link: geometry collision mesh filename=package://hpp_environments/meshes/multicontact/daeun/bridge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; visual mesh filename=package://hpp_environments/meshes/multicontact/daeun/bridge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

File: urdf/multicontact/daeun/rubbles_1.urdf (robot description, URDF)
Before this commit: robot rubbles_1, 1 links, 0 joints
Links:
- link base_link: geometry collision mesh filename=package://hpp_environments/meshes/multicontact/daeun/rubble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; visual mesh filename=package://hpp_environments/meshes/multicontact/daeun/rubble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

File: urdf/multicontact/daeun/rubbles_2.urdf (robot description, URDF)
Before this commit: robot rubbles_2, 1 links, 0 joints
Links:
- link base_link: geometry collision mesh filename=package://hpp_environments/meshes/multicontact/daeun/rubble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; visual mesh filename=package://hpp_environments/meshes/multicontact/daeun/rubble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

File: urdf/multicontact/daeun/rubbles_3.urdf (robot description, URDF)
Before this commit: robot rubbles_3, 1 links, 0 joints
Links:
- link base_link: geometry collision mesh filename=package://hpp_environments/meshes/multicontact/daeun/rubble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; visual mesh filename=package://hpp_environments/meshes/multicontact/daeun/rubble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

File: urdf/multicontact/daeun/rubbles_4.urdf (robot description, URDF)
Before this commit: robot rubbles_4, 1 links, 0 joints
Links:
- link base_link: geometry collision mesh filename=package://hpp_environments/meshes/multicontact/daeun/rubble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; visual mesh filename=package://hpp_environments/meshes/multicontact/daeun/rubble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

File: urdf/multicontact/daeun/rubbles_5.urdf (robot description, URDF)
Before this commit: robot rubbles_5, 1 links, 0 joints
Links:
- link base_link: geometry collision mesh filename=package://hpp_environments/meshes/multicontact/daeun/rubble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; visual mesh filename=package://hpp_environments/meshes/multicontact/daeun/rubble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

File: urdf/multicontact/daeun/rubbles_6.urdf (robot description, URDF)
Before this commit: robot rubbles_6, 1 links, 0 joints
Links:
- link base_link: geometry collision mesh filename=package://hpp_environments/meshes/multicontact/daeun/rubble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; visual mesh filename=package://hpp_environments/meshes/multicontact/daeun/rubble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

File: urdf/multicontact/daeun/rubbles_7.urdf (robot description, URDF)
Before this commit: robot rubbles_7, 1 links, 0 joints
Links:
- link base_link: geometry collision mesh filename=package://hpp_environments/meshes/multicontact/daeun/rubble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; visual mesh filename=package://hpp_environments/meshes/multicontact/daeun/rubble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

File: urdf/multicontact/daeun/rubbles_stairs_1.urdf (robot description, URDF)
Before this commit: robot rubbles_stairs_1, 1 links, 0 joints
Links:
- link base_link: geometry collision mesh filename=package://hpp_environments/meshes/multicontact/daeun/rubble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; visual mesh filename=package://hpp_environments/meshes/multicontact/daeun/rubble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

File: urdf/multicontact/daeun/rubbles_stairs_2.urdf (robot description, URDF)
Before this commit: robot rubbles_stairs_2, 1 links, 0 joints
Links:
- link base_link: geometry collision mesh filename=package://hpp_environments/meshes/multicontact/daeun/rubble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; visual mesh filename=package://hpp_environments/meshes/multicontact/daeun/rubble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

File: urdf/multicontact/daeun/rubbles_stairs_3.urdf (robot description, URDF)
Before this commit: robot rubbles_stairs_3, 1 links, 0 joints
Links:
- link base_link: geometry collision mesh filename=package://hpp_environments/meshes/multicontact/daeun/rubble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; visual mesh filename=package://hpp_environments/meshes/multicontact/daeun/rubble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

File: urdf/multicontact/daeun/rubbles_stairs_bridge_1.urdf (robot description, URDF)
Before this commit: robot rubbles_stairs_bridge_1, 1 links, 0 joints
Links:
- link base_link: geometry collision mesh filename=package://hpp_environments/meshes/multicontact/daeun/rubble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; visual mesh filename=package://hpp_environments/meshes/multicontact/daeun/rubble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

File: urdf/multicontact/daeun/rubbles_stairs_bridge_2.urdf (robot description, URDF)
Before this commit: robot rubbles_stairs_bridge_2, 1 links, 0 joints
Links:
- link base_link: geometry collision mesh filename=package://hpp_environments/meshes/multicontact/daeun/rubble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; visual mesh filename=package://hpp_environments/meshes/multicontact/daeun/rubble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

File: urdf/multicontact/daeun/stairs_1.urdf (robot description, URDF)
Before this commit: robot stairs_1, 1 links, 0 joints
Links:
- link base_link: geometry collision mesh filename=package://hpp_environments/meshes/multicontact/daeun/stairs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; visual mesh filename=package://hpp_environments/meshes/multicontact/daeun/stairs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

File: urdf/multicontact/daeun/stairs_2.urdf (robot description, URDF)
Before this commit: robot stairs_2, 1 links, 0 joints
Links:
- link base_link: geometry collision mesh filename=package://hpp_environments/meshes/multicontact/daeun/stairs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; visual mesh filename=package://hpp_environments/meshes/multicontact/daeun/stairs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

File: urdf/multicontact/daeun/stairs_3.urdf (robot description, URDF)
Before this commit: robot stairs_3, 1 links, 0 joints
Links:
- link base_link: geometry collision mesh filename=package://hpp_environments/meshes/multicontact/daeun/stairs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; visual mesh filename=package://hpp_environments/meshes/multicontact/daeun/stairs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

File: urdf/multicontact/daeun/stairs_bridge_1.urdf (robot description, URDF)
Before this commit: robot stairs_bridge_1, 1 links, 0 joints
Links:
- link base_link: geometry collision mesh filename=package://hpp_environments/meshes/multicontact/daeun/stairs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; visual mesh filename=package://hpp_environments/meshes/multicontact/daeun/stairs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

File: urdf/multicontact/daeun/stairs_bridge_2.urdf (robot description, URDF)
Before this commit: robot stairs_bridge_2, 1 links, 0 joints
Links:
- link base_link: geometry collision mesh filename=package://hpp_environments/meshes/multicontact/daeun/stairs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; visual mesh filename=package://hpp_environments/meshes/multicontact/daeun/stairs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
